File: TP-Board-iso105.kicad_sch (KiCad schematic)
At the start: 437 parts, among them SW1 SW_Push, SW10 SW_Push, SW100 SW_Push, SW101 SW_Push, SW102 SW_Push, SW103 SW_Push, SW104 SW_Push, SW105 SW_Push, SW106 SW_Push, SW107 SW_Push, SW108 SW_Push, SW109 SW_Push, SW11 SW_Push, SW12 SW_Push, SW13 SW_Push, SW14 SW_Push, SW15 SW_Push, SW16 SW_Push, SW17 SW_Push, SW18 SW_Push, SW19 SW_Push, SW2 SW_Push, SW20 SW_Push, SW21 SW_Push, SW22 SW_Push, SW23 SW_Push, SW24 SW_Push, SW25 SW_Push, SW26 SW_Push, SW27 SW_Push, SW28 SW_Push, SW29 SW_Push, SW3 SW_Push, SW30 SW_Push, SW31 SW_Push, SW32 SW_Push, SW33 SW_Push, SW34 SW_Push, SW35 SW_Push, SW36 SW_Push, SW37 SW_Push, SW38 SW_Push, SW39 SW_Push, SW4 SW_Push, SW40 SW_Push, SW41 SW_Push, SW42 SW_Push, SW43 SW_Push, SW44 SW_Push, SW45 SW_Push, SW46 SW_Push, SW47 SW_Push, SW48 SW_Push, SW49 SW_Push, SW5 SW_Push, SW50 SW_Push, SW51 SW_Push, SW52 SW_Push, SW53 SW_Push, SW54 SW_Push, SW55 SW_Push, SW56 SW_Push, SW57 SW_Push, SW58 SW_Push, SW59 SW_Push, SW6 SW_Push, SW60 SW_Push, SW61 SW_Push, SW62 SW_Push, SW63 SW_Push, SW64 SW_Push, SW65 SW_Push, SW66 SW_Push, SW67 SW_Push, SW68 SW_Push, SW69 SW_Push, SW7 SW_Push, SW70 SW_Push, SW71 SW_Push, SW72 SW_Push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

Commit message: 👌
Parts:
- removed D110, D112, D113, D114, D115, D116, D117, D118, D119, D120, D121, D122, D123, D124, D125, D126, D127, D128, D129, D130, D131, D132, D133, D134, D135, D136, D137, D138, D139, D140, D141, D142, D143, D144, D145, D146, D147, D148, D149, D150, D151, D152, D153, D154, D155, D156, D157, D158, D159, D160, D161, D162, D163, D164, D165, D166, D167, D168, D169, D170, D171, D172, D173, D174, D175, D176, D177, D178, D179, D180, D181, D182, D183, D184, D185, D186, D187, D188, D189, D190, D191, D192, D193, D194, D195, D196, D197, D198, D199, D200, D201, D202, D203, D204, D205, D206, D207, D208, D209, D210, D211, D212, D213, D214, D215, D216, D217, D218: IR26-21C_L110_TR8, LED_SMD:LED_1206_3216Metric, symbol LED:IR26-21C_L110_TR8
- removed D111: IR26-21C_L110_TR8, LED_SMD:LED_0201_0603Metric, symbol LED:IR26-21C_L110_TR8
- removed D17, D18, D19, D20: 1N4148, Diode_SMD:D_SOD-323F, symbol Diode:1N4148
- removed R106, R107, R108, R109: 68, Resistor_SMD:R_0201_0603Metric, symbol Device:R
- removed SW17, SW18, SW19, SW20: SW_Push, Scotto:Gateron_Low_Profile_Socket, symbol Switch:SW_Push
- added H1, H2, H3, H4: Mounting_Hole, MountingHole:MountingHole_2.2mm_M2_DIN965, symbol Scotto:Placeholder_Mounting_Hole
- added LED1, LED10, LED100, LED101, LED102, LED103, LED104, LED105, LED11, LED12, LED13, LED14, LED15, LED16, LED17, LED18, LED19, LED2, LED20, LED21, LED22, LED23, LED24, LED25, LED26, LED27, LED28, LED29, LED3, LED30, LED31, LED32, LED33, LED34, LED35, LED36, LED37, LED38, LED39, LED4, LED40, LED41, LED42, LED43, LED44, LED45, LED46, LED47, LED48, LED49, LED5, LED50, LED51, LED52, LED53, LED54, LED55, LED56, LED57, LED58, LED59, LED6, LED60, LED61, LED62, LED63, LED64, LED65, LED66, LED67, LED68, LED69, LED7, LED70, LED71, LED72, LED73, LED74, LED75, LED76, LED77, LED78, LED79, LED8, LED80, LED81, LED82, LED83, LED84, LED85, LED86, LED87, LED88, LED89, LED9, LED90, LED91, LED92, LED93, LED94, LED95, LED96, LED97, LED98, LED99: LSM0603443V, LED_SMD:LED_0603_1608Metric, symbol Scotto:Placeholder_LED
- D1, D10, D11, D12, D13, D14, D15, D16, D2, D3, D4, D5, D6, D7, D8, D9: value 1N4148 -> 1N4148WT; footprint Diode_SMD:D_SOD-323F -> Diode_SMD:D_SOD-523
- D100: renamed from D104; value 1N4148 -> 1N4148WT; footprint Diode_SMD:D_SOD-323F -> Diode_SMD:D_SOD-523
- D101: renamed from D105; value 1N4148 -> 1N4148WT; footprint Diode_SMD:D_SOD-323F -> Diode_SMD:D_SOD-523
- D102: renamed from D106; value 1N4148 -> 1N4148WT; footprint Diode_SMD:D_SOD-323F -> Diode_SMD:D_SOD-523
- D103: renamed from D107; value 1N4148 -> 1N4148WT; footprint Diode_SMD:D_SOD-323F -> Diode_SMD:D_SOD-523
- D104: renamed from D108; value 1N4148 -> 1N4148WT; footprint Diode_SMD:D_SOD-323F -> Diode_SMD:D_SOD-523
- D105: renamed from D109; value 1N4148 -> 1N4148WT; footprint Diode_SMD:D_SOD-323F -> Diode_SMD:D_SOD-523
- D17: renamed from D21; value 1N4148 -> 1N4148WT; footprint Diode_SMD:D_SOD-323F -> Diode_SMD:D_SOD-523
- D18: renamed from D22; value 1N4148 -> 1N4148WT; footprint Diode_SMD:D_SOD-323F -> Diode_SMD:D_SOD-523
- D19: renamed from D23; value 1N4148 -> 1N4148WT; footprint Diode_SMD:D_SOD-323F -> Diode_SMD:D_SOD-523
- D20: renamed from D24; value 1N4148 -> 1N4148WT; footprint Diode_SMD:D_SOD-323F -> Diode_SMD:D_SOD-523
- D21: renamed from D25; value 1N4148 -> 1N4148WT; footprint Diode_SMD:D_SOD-323F -> Diode_SMD:D_SOD-523
- D22: renamed from D26; value 1N4148 -> 1N4148WT; footprint Diode_SMD:D_SOD-323F -> Diode_SMD:D_SOD-523
- D23: renamed from D27; value 1N4148 -> 1N4148WT; footprint Diode_SMD:D_SOD-323F -> Diode_SMD:D_SOD-523
- D24: renamed from D28; value 1N4148 -> 1N4148WT; footprint Diode_SMD:D_SOD-323F -> Diode_SMD:D_SOD-523
- D25: renamed from D29; value 1N4148 -> 1N4148WT; footprint Diode_SMD:D_SOD-323F -> Diode_SMD:D_SOD-523
- D26: renamed from D30; value 1N4148 -> 1N4148WT; footprint Diode_SMD:D_SOD-323F -> Diode_SMD:D_SOD-523
- D27: renamed from D31; value 1N4148 -> 1N4148WT; footprint Diode_SMD:D_SOD-323F -> Diode_SMD:D_SOD-523
- D28: renamed from D32; value 1N4148 -> 1N4148WT; footprint Diode_SMD:D_SOD-323F -> Diode_SMD:D_SOD-523
- D29: renamed from D33; value 1N4148 -> 1N4148WT; footprint Diode_SMD:D_SOD-323F -> Diode_SMD:D_SOD-523
- D30: renamed from D34; value 1N4148 -> 1N4148WT; footprint Diode_SMD:D_SOD-323F -> Diode_SMD:D_SOD-523
- D31: renamed from D35; value 1N4148 -> 1N4148WT; footprint Diode_SMD:D_SOD-323F -> Diode_SMD:D_SOD-523
- D32: renamed from D36; value 1N4148 -> 1N4148WT; footprint Diode_SMD:D_SOD-323F -> Diode_SMD:D_SOD-523
- D33: renamed from D37; value 1N4148 -> 1N4148WT; footprint Diode_SMD:D_SOD-323F -> Diode_SMD:D_SOD-523
- D34: renamed from D38; value 1N4148 -> 1N4148WT; footprint Diode_SMD:D_SOD-323F -> Diode_SMD:D_SOD-523
- D35: renamed from D39; value 1N4148 -> 1N4148WT; footprint Diode_SMD:D_SOD-323F -> Diode_SMD:D_SOD-523
- D36: renamed from D40; value 1N4148 -> 1N4148WT; footprint Diode_SMD:D_SOD-323F -> Diode_SMD:D_SOD-523
- D37: renamed from D41; value 1N4148 -> 1N4148WT; footprint Diode_SMD:D_SOD-323F -> Diode_SMD:D_SOD-523
- D38: renamed from D42; value 1N4148 -> 1N4148WT; footprint Diode_SMD:D_SOD-323F -> Diode_SMD:D_SOD-523
- D39: renamed from D43; value 1N4148 -> 1N4148WT; footprint Diode_SMD:D_SOD-323F -> Diode_SMD:D_SOD-523
- D40: renamed from D44; value 1N4148 -> 1N4148WT; footprint Diode_SMD:D_SOD-323F -> Diode_SMD:D_SOD-523
- D41: renamed from D45; value 1N4148 -> 1N4148WT; footprint Diode_SMD:D_SOD-323F -> Diode_SMD:D_SOD-523
- D42: renamed from D46; value 1N4148 -> 1N4148WT; footprint Diode_SMD:D_SOD-323F -> Diode_SMD:D_SOD-523
- D43: renamed from D47; value 1N4148 -> 1N4148WT; footprint Diode_SMD:D_SOD-323F -> Diode_SMD:D_SOD-523
- D44: renamed from D48; value 1N4148 -> 1N4148WT; footprint Diode_SMD:D_SOD-323F -> Diode_SMD:D_SOD-523
- D45: renamed from D49; value 1N4148 -> 1N4148WT; footprint Diode_SMD:D_SOD-323F -> Diode_SMD:D_SOD-523
- D46: renamed from D50; value 1N4148 -> 1N4148WT; footprint Diode_SMD:D_SOD-323F -> Diode_SMD:D_SOD-523
- D47: renamed from D51; value 1N4148 -> 1N4148WT; footprint Diode_SMD:D_SOD-323F -> Diode_SMD:D_SOD-523
- D48: renamed from D52; value 1N4148 -> 1N4148WT; footprint Diode_SMD:D_SOD-323F -> Diode_SMD:D_SOD-523
- D49: renamed from D53; value 1N4148 -> 1N4148WT; footprint Diode_SMD:D_SOD-323F -> Diode_SMD:D_SOD-523
- D50: renamed from D54; value 1N4148 -> 1N4148WT; footprint Diode_SMD:D_SOD-323F -> Diode_SMD:D_SOD-523
- D51: renamed from D55; value 1N4148 -> 1N4148WT; footprint Diode_SMD:D_SOD-323F -> Diode_SMD:D_SOD-523
- D52: renamed from D56; value 1N4148 -> 1N4148WT; footprint Diode_SMD:D_SOD-323F -> Diode_SMD:D_SOD-523
- D53: renamed from D57; value 1N4148 -> 1N4148WT; footprint Diode_SMD:D_SOD-323F -> Diode_SMD:D_SOD-523
- D54: renamed from D58; value 1N4148 -> 1N4148WT; footprint Diode_SMD:D_SOD-323F -> Diode_SMD:D_SOD-523
- D55: renamed from D59; value 1N4148 -> 1N4148WT; footprint Diode_SMD:D_SOD-323F -> Diode_SMD:D_SOD-523
- D56: renamed from D60; value 1N4148 -> 1N4148WT; footprint Diode_SMD:D_SOD-323F -> Diode_SMD:D_SOD-523
- D57: renamed from D61; value 1N4148 -> 1N4148WT; footprint Diode_SMD:D_SOD-323F -> Diode_SMD:D_SOD-523
- D58: renamed from D62; value 1N4148 -> 1N4148WT; footprint Diode_SMD:D_SOD-323F -> Diode_SMD:D_SOD-523
- D59: renamed from D63; value 1N4148 -> 1N4148WT; footprint Diode_SMD:D_SOD-323F -> Diode_SMD:D_SOD-523
- D60: renamed from D64; value 1N4148 -> 1N4148WT; footprint Diode_SMD:D_SOD-323F -> Diode_SMD:D_SOD-523
- D61: renamed from D65; value 1N4148 -> 1N4148WT; footprint Diode_SMD:D_SOD-323F -> Diode_SMD:D_SOD-523
- D62: renamed from D66; value 1N4148 -> 1N4148WT; footprint Diode_SMD:D_SOD-323F -> Diode_SMD:D_SOD-523
- D63: renamed from D67; value 1N4148 -> 1N4148WT; footprint Diode_SMD:D_SOD-323F -> Diode_SMD:D_SOD-523
- D64: renamed from D68; value 1N4148 -> 1N4148WT; footprint Diode_SMD:D_SOD-323F -> Diode_SMD:D_SOD-523
- D65: renamed from D69; value 1N4148 -> 1N4148WT; footprint Diode_SMD:D_SOD-323F -> Diode_SMD:D_SOD-523
- D66: renamed from D70; value 1N4148 -> 1N4148WT; footprint Diode_SMD:D_SOD-323F -> Diode_SMD:D_SOD-523
- D67: renamed from D71; value 1N4148 -> 1N4148WT; footprint Diode_SMD:D_SOD-323F -> Diode_SMD:D_SOD-523
- D68: renamed from D72; value 1N4148 -> 1N4148WT; footprint Diode_SMD:D_SOD-323F -> Diode_SMD:D_SOD-523
- D69: renamed from D73; value 1N4148 -> 1N4148WT; footprint Diode_SMD:D_SOD-323F -> Diode_SMD:D_SOD-523
- D70: renamed from D74; value 1N4148 -> 1N4148WT; footprint Diode_SMD:D_SOD-323F -> Diode_SMD:D_SOD-523
- D71: renamed from D75; value 1N4148 -> 1N4148WT; footprint Diode_SMD:D_SOD-323F -> Diode_SMD:D_SOD-523
- D72: renamed from D76; value 1N4148 -> 1N4148WT; footprint Diode_SMD:D_SOD-323F -> Diode_SMD:D_SOD-523
- D73: renamed from D77; value 1N4148 -> 1N4148WT; footprint Diode_SMD:D_SOD-323F -> Diode_SMD:D_SOD-523
- D74: renamed from D78; value 1N4148 -> 1N4148WT; footprint Diode_SMD:D_SOD-323F -> Diode_SMD:D_SOD-523
- D75: renamed from D79; value 1N4148 -> 1N4148WT; footprint Diode_SMD:D_SOD-323F -> Diode_SMD:D_SOD-523
- D76: renamed from D80; value 1N4148 -> 1N4148WT; footprint Diode_SMD:D_SOD-323F -> Diode_SMD:D_SOD-523
- D77: renamed from D81; value 1N4148 -> 1N4148WT; footprint Diode_SMD:D_SOD-323F -> Diode_SMD:D_SOD-523
- D78: renamed from D82; value 1N4148 -> 1N4148WT; footprint Diode_SMD:D_SOD-323F -> Diode_SMD:D_SOD-523
- D79: renamed from D83; value 1N4148 -> 1N4148WT; footprint Diode_SMD:D_SOD-323F -> Diode_SMD:D_SOD-523
- D80: renamed from D84; value 1N4148 -> 1N4148WT; footprint Diode_SMD:D_SOD-323F -> Diode_SMD:D_SOD-523
- D81: renamed from D85; value 1N4148 -> 1N4148WT; footprint Diode_SMD:D_SOD-323F -> Diode_SMD:D_SOD-523
- D82: renamed from D86; value 1N4148 -> 1N4148WT; footprint Diode_SMD:D_SOD-323F -> Diode_SMD:D_SOD-523
- D83: renamed from D87; value 1N4148 -> 1N4148WT; footprint Diode_SMD:D_SOD-323F -> Diode_SMD:D_SOD-523
- D84: renamed from D88; value 1N4148 -> 1N4148WT; footprint Diode_SMD:D_SOD-323F -> Diode_SMD:D_SOD-523
- D85: renamed from D89; value 1N4148 -> 1N4148WT; footprint Diode_SMD:D_SOD-323F -> Diode_SMD:D_SOD-523
- D86: renamed from D90; value 1N4148 -> 1N4148WT; footprint Diode_SMD:D_SOD-323F -> Diode_SMD:D_SOD-523
- D87: renamed from D91; value 1N4148 -> 1N4148WT; footprint Diode_SMD:D_SOD-323F -> Diode_SMD:D_SOD-523
- D88: renamed from D92; value 1N4148 -> 1N4148WT; footprint Diode_SMD:D_SOD-323F -> Diode_SMD:D_SOD-523
- D89: renamed from D93; value 1N4148 -> 1N4148WT; footprint Diode_SMD:D_SOD-323F -> Diode_SMD:D_SOD-523
- D90: renamed from D94; value 1N4148 -> 1N4148WT; footprint Diode_SMD:D_SOD-323F -> Diode_SMD:D_SOD-523
- D91: renamed from D95; value 1N4148 -> 1N4148WT; footprint Diode_SMD:D_SOD-323F -> Diode_SMD:D_SOD-523
- D92: renamed from D96; value 1N4148 -> 1N4148WT; footprint Diode_SMD:D_SOD-323F -> Diode_SMD:D_SOD-523
- D93: renamed from D97; value 1N4148 -> 1N4148WT; footprint Diode_SMD:D_SOD-323F -> Diode_SMD:D_SOD-523
- D94: renamed from D98; value 1N4148 -> 1N4148WT; footprint Diode_SMD:D_SOD-323F -> Diode_SMD:D_SOD-523
- D95: renamed from D99; value 1N4148 -> 1N4148WT; footprint Diode_SMD:D_SOD-323F -> Diode_SMD:D_SOD-523
- D96: renamed from D100; value 1N4148 -> 1N4148WT; footprint Diode_SMD:D_SOD-323F -> Diode_SMD:D_SOD-523
- D97: renamed from D101; value 1N4148 -> 1N4148WT; footprint Diode_SMD:D_SOD-323F -> Diode_SMD:D_SOD-523
- D98: renamed from D102; value 1N4148 -> 1N4148WT; footprint Diode_SMD:D_SOD-323F -> Diode_SMD:D_SOD-523
- D99: renamed from D103; value 1N4148 -> 1N4148WT; footprint Diode_SMD:D_SOD-323F -> Diode_SMD:D_SOD-523
- R1, R10, R100, R101, R102, R103, R104, R105, R11, R12, R13, R14, R15, R16, R17, R18, R19, R2, R20, R21, R22, R23, R24, R25, R26, R27, R28, R29, R3, R30, R31, R32, R33, R34, R35, R36, R37, R38, R39, R4, R40, R41, R42, R43, R44, R45, R46, R47, R48, R49, R5, R50, R51, R52, R53, R54, R55, R56, R57, R58, R59, R6, R60, R61, R62, R63, R64, R65, R66, R67, R68, R69, R7, R70, R71, R72, R73, R74, R75, R76, R77, R78, R79, R8, R80, R81, R82, R83, R84, R85, R86, R87, R88, R89, R9, R90, R91, R92, R93, R94, R95, R96, R97, R98, R99: value 68 -> 150; footprint Resistor_SMD:R_0201_0603Metric -> Resistor_SMD:R_0201_0603Metric_Pad0.64x0.40mm_HandSolder
- U1: footprint ScottoKeebs_MCU:Raspberry_Pi_Pico -> ScottoKeebs_MCU:Raspberry_Pi_Pico_2W
- renumbered SW104 to SW100, SW105 to SW101, SW106 to SW102, SW107 to SW103, SW108 to SW104, SW109 to SW105, SW21 to SW17, SW22 to SW18, SW23 to SW19, SW24 to SW20, SW25 to SW21, SW26 to SW22, SW27 to SW23, SW28 to SW24, SW29 to SW25, SW30 to SW26, SW31 to SW27, SW32 to SW28, SW33 to SW29, SW34 to SW30, SW35 to SW31, SW36 to SW32, SW37 to SW33, SW38 to SW34, SW39 to SW35, SW40 to SW36, SW41 to SW37, SW42 to SW38, SW43 to SW39, SW44 to SW40, SW45 to SW41, SW46 to SW42, SW47 to SW43, SW48 to SW44, SW49 to SW45, SW50 to SW46, SW51 to SW47, SW52 to SW48, SW53 to SW49, SW54 to SW50, SW55 to SW51, SW56 to SW52, SW57 to SW53, SW58 to SW54, SW59 to SW55, SW60 to SW56, SW61 to SW57, SW62 to SW58, SW63 to SW59, SW64 to SW60, SW65 to SW61, SW66 to SW62, SW67 to SW63, SW68 to SW64, SW69 to SW65, SW70 to SW66, SW71 to SW67, SW72 to SW68, SW73 to SW69, SW74 to SW70, SW75 to SW71, SW76 to SW72, SW77 to SW73, SW78 to SW74, SW79 to SW75, SW80 to SW76, SW81 to SW77, SW82 to SW78, SW83 to SW79, SW84 to SW80, SW85 to SW81, SW86 to SW82, SW87 to SW83, SW88 to SW84, SW89 to SW85, SW90 to SW86, SW91 to SW87, SW92 to SW88, SW93 to SW89, SW94 to SW90, SW95 to SW91, SW96 to SW92, SW97 to SW93, SW98 to SW94, SW99 to SW95, SW100 to SW96, SW101 to SW97, SW102 to SW98, SW103 to SW99
Connections:
- net COL0: now also SW34.1; no longer SW89.1
- net COL1: now also SW35.1; no longer SW90.1
- net COL10: now also SW74.1; no longer SW57.1
- net COL11: now also SW89.1; no longer SW58.1
- net COL12: now also SW90.1; no longer SW72.1
- net COL13: now also SW91.1; no longer SW73.1
- net COL14: now also SW92.1; no longer SW74.1
- net COL15: now also SW104.1
- net COL16: now also SW105.1
- net COL2: now also SW36.1; no longer SW91.1
- net COL3: now also SW37.1; no longer SW92.1
- net COL4: now also SW55.1; no longer SW104.1, SW34.1
- net COL5: now also SW56.1; no longer SW105.1, SW35.1
- net COL6: now also SW57.1; no longer SW36.1
- net COL7: now also SW58.1; no longer SW37.1
- net COL8: now also SW72.1; no longer SW55.1
- net COL9: now also SW73.1; no longer SW56.1
- net ROW6: now also D104.1 (K), D105.1 (K), D89.1 (K), D90.1 (K), D91.1 (K), D92.1 (K), U1.9 (GPIO6); no longer U1.8 (GND)
- net ROW7: now also U1.10 (GPIO7); no longer D104.1 (K), D105.1 (K), D89.1 (K), D90.1 (K), D91.1 (K), D92.1 (K), U1.9 (GPIO6)
- net at R103.1: now also LED103.2 (A)
- net at R76.1: now also LED76.2 (A)
- net at R44.1: now also LED44.2 (A)
- net at R42.1: now also LED42.2 (A)
- net at R67.1: now also LED67.2 (A)
- net at R17.1: now also LED17.2 (A)
- net at R1.1: now also LED1.2 (A)
- net at R74.1: now also LED74.2 (A)
- net at R78.1: now also LED78.2 (A)
- net at R22.1: now also LED22.2 (A)
- net at R29.1: now also LED29.2 (A)
- net at R20.1: now also LED20.2 (A)
- net at R72.1: now also LED72.2 (A)
- net at R82.1: now also LED82.2 (A)
- net at R43.1: now also LED43.2 (A)
- net at R81.1: now also LED81.2 (A)
- net at R31.1: now also LED31.2 (A)
- net at R49.1: now also LED49.2 (A)
- net at R11.1: now also LED11.2 (A)
- net at R12.1: now also LED12.2 (A)
- net at R88.1: now also LED88.2 (A)
- net at R97.1: now also LED97.2 (A)
- net at R86.1: now also LED86.2 (A)
- net at R100.1: now also LED100.2 (A)
- net at R73.1: now also LED73.2 (A)
- net at R14.1: now also LED14.2 (A)
- net at R95.1: now also LED95.2 (A)
- net at R69.1: now also LED69.2 (A)
- net at R70.1: now also LED70.2 (A)
- net at R64.1: now also LED64.2 (A)
- net at R23.1: now also LED23.2 (A)
- net at R46.1: now also LED46.2 (A)
- net at R41.1: now also LED41.2 (A)
- net at R80.1: now also LED80.2 (A)
- net at R59.1: now also LED59.2 (A)
- net at R4.1: now also LED4.2 (A)
- net at R9.1: now also LED9.2 (A)
- net at R54.1: now also LED54.2 (A)
- net at R30.1: now also LED30.2 (A)
- net at R104.1: now also LED104.2 (A)
- net at R27.1: now also LED27.2 (A)
- net at R15.1: now also LED15.2 (A)
- net at R18.1: now also LED18.2 (A)
- net at R79.1: now also LED79.2 (A)
- net at R63.1: now also LED63.2 (A)
- net at R96.1: now also LED96.2 (A)
- net at R65.1: now also LED65.2 (A)
- net at R87.1: now also LED87.2 (A)
- net at R94.1: now also LED94.2 (A)
- net at R56.1: now also LED56.2 (A)
- net at R101.1: now also LED101.2 (A)
- net at R40.1: now also LED40.2 (A)
- net at R89.1: now also LED89.2 (A)
- net at R105.1: now also LED105.2 (A)
- net at R10.1: now also LED10.2 (A)
- net at R57.1: now also LED57.2 (A)
- net at R28.1: now also LED28.2 (A)
- net at R75.1: now also LED75.2 (A)
- net at R6.1: now also LED6.2 (A)
- net at R26.1: now also LED26.2 (A)
- net at R68.1: now also LED68.2 (A)
- net at R24.1: now also LED24.2 (A)
- net at R35.1: now also LED35.2 (A)
- net at R102.1: now also LED102.2 (A)
- net at R53.1: now also LED53.2 (A)
- net at R37.1: now also LED37.2 (A)
- net at R71.1: now also LED71.2 (A)
- net at R33.1: now also LED33.2 (A)
- net at R58.1: now also LED58.2 (A)
- net at R84.1: now also LED84.2 (A)
- net at R83.1: now also LED83.2 (A)
- net at R93.1: now also LED93.2 (A)
- net at R77.1: now also LED77.2 (A)
- net at R50.1: now also LED50.2 (A)
- net at R98.1: now also LED98.2 (A)
- net at R47.1: now also LED47.2 (A)
- net at R19.1: now also LED19.2 (A)
- net at R52.1: now also LED52.2 (A)
- net at R16.1: now also LED16.2 (A)
- net at R51.1: now also LED51.2 (A)
- net at R48.1: now also LED48.2 (A)
- net at R25.1: now also LED25.2 (A)
- net at R55.1: now also LED55.2 (A)
- net at R85.1: now also LED85.2 (A)
- net at R66.1: now also LED66.2 (A)
- net at R5.1: now also LED5.2 (A)
- net at R62.1: now also LED62.2 (A)
- net at R2.1: now also LED2.2 (A)
- net at R61.1: now also LED61.2 (A)
- net at R32.1: now also LED32.2 (A)
- net at R8.1: now also LED8.2 (A)
- net at R3.1: now also LED3.2 (A)
- net at R21.1: now also LED21.2 (A)
- net at R36.1: now also LED36.2 (A)
- net at R91.1: now also LED91.2 (A)
- net at R7.1: now also LED7.2 (A)
- net at R39.1: now also LED39.2 (A)
- net at R38.1: now also LED38.2 (A)
- net at R92.1: now also LED92.2 (A)
- net at R90.1: now also LED90.2 (A)
- net at R34.1: now also LED34.2 (A)
- net at R13.1: now also LED13.2 (A)
- net at R60.1: now also LED60.2 (A)
- net at R99.1: now also LED99.2 (A)
- net at R45.1: now also LED45.2 (A)
- new net GND: LED1.1 (K), LED10.1 (K), LED100.1 (K), LED101.1 (K), LED102.1 (K), LED103.1 (K), LED104.1 (K), LED105.1 (K), LED11.1 (K), LED12.1 (K), LED13.1 (K), LED14.1 (K), LED15.1 (K), LED16.1 (K), LED17.1 (K), LED18.1 (K), LED19.1 (K), LED2.1 (K), LED20.1 (K), LED21.1 (K), LED22.1 (K), LED23.1 (K), LED24.1 (K), LED25.1 (K), LED26.1 (K), LED27.1 (K), LED28.1 (K), LED29.1 (K), LED3.1 (K), LED30.1 (K), LED31.1 (K), LED32.1 (K), LED33.1 (K), LED34.1 (K), LED35.1 (K), LED36.1 (K), LED37.1 (K), LED38.1 (K), LED39.1 (K), LED4.1 (K), LED40.1 (K), LED41.1 (K), LED42.1 (K), LED43.1 (K), LED44.1 (K), LED45.1 (K), LED46.1 (K), LED47.1 (K), LED48.1 (K), LED49.1 (K), LED5.1 (K), LED50.1 (K), LED51.1 (K), LED52.1 (K), LED53.1 (K), LED54.1 (K), LED55.1 (K), LED56.1 (K), LED57.1 (K), LED58.1 (K), LED59.1 (K), LED6.1 (K), LED60.1 (K), LED61.1 (K), LED62.1 (K), LED63.1 (K), LED64.1 (K), LED65.1 (K), LED66.1 (K), LED67.1 (K), LED68.1 (K), LED69.1 (K), LED7.1 (K), LED70.1 (K), LED71.1 (K), LED72.1 (K), LED73.1 (K), LED74.1 (K), LED75.1 (K), LED76.1 (K), LED77.1 (K), LED78.1 (K), LED79.1 (K), LED8.1 (K), LED80.1 (K), LED81.1 (K), LED82.1 (K), LED83.1 (K), LED84.1 (K), LED85.1 (K), LED86.1 (K), LED87.1 (K), LED88.1 (K), LED89.1 (K), LED9.1 (K), LED90.1 (K), LED91.1 (K), LED92.1 (K), LED93.1 (K), LED94.1 (K), LED95.1 (K), LED96.1 (K), LED97.1 (K), LED98.1 (K), LED99.1 (K), U1.8 (GND)

Commit message: 💀
Parts:
- H1, H2, H3, H4, SW1, SW10, SW100, SW101, SW102, SW103, SW104, SW105, SW11, SW12, SW13, SW14, SW15, SW16, SW17, SW18, SW19, SW2, SW20, SW21, SW22, SW23, SW24, SW25, SW26, SW27, SW28, SW29, SW3, SW30, SW31, SW32, SW33, SW34, SW35, SW36, SW37, SW38, SW39, SW4, SW40, SW41, SW42, SW43, SW44, SW45, SW46, SW47, SW48, SW49, SW5, SW50, SW51, SW52, SW53, SW54, SW55, SW56, SW57, SW58, SW59, SW6, SW60, SW61, SW62, SW63, SW64, SW65, SW66, SW67, SW68, SW69, SW7, SW70, SW71, SW72, SW73, SW74, SW75, SW76, SW77, SW78, SW79, SW8, SW80, SW81, SW82, SW83, SW84, SW85, SW86, SW87, SW88, SW89, SW9, SW90, SW91, SW92, SW93, SW94, SW95, SW96, SW97, SW98, SW99, U1: now left out of the parts list
- LED1, LED10, LED100, LED101, LED102, LED103, LED104, LED105, LED11, LED12, LED13, LED14, LED15, LED16, LED17, LED18, LED19, LED2, LED20, LED21, LED22, LED23, LED24, LED25, LED26, LED27, LED28, LED29, LED3, LED30, LED31, LED32, LED33, LED34, LED35, LED36, LED37, LED38, LED39, LED4, LED40, LED41, LED42, LED43, LED44, LED45, LED46, LED47, LED48, LED49, LED5, LED50, LED51, LED52, LED53, LED54, LED55, LED56, LED57, LED58, LED59, LED6, LED60, LED61, LED62, LED63, LED64, LED65, LED66, LED67, LED68, LED69, LED7, LED70, LED71, LED72, LED73, LED74, LED75, LED76, LED77, LED78, LED79, LED8, LED80, LED81, LED82, LED83, LED84, LED85, LED86, LED87, LED88, LED89, LED9, LED90, LED91, LED92, LED93, LED94, LED95, LED96, LED97, LED98, LED99: value LSM0603443V -> XL-1608UWC-04
- R1, R10, R100, R101, R102, R103, R104, R105, R11, R12, R13, R14, R15, R16, R17, R18, R19, R2, R20, R21, R22, R23, R24, R25, R26, R27, R28, R29, R3, R30, R31, R32, R33, R34, R35, R36, R37, R38, R39, R4, R40, R41, R42, R43, R44, R45, R46, R47, R48, R49, R5, R50, R51, R52, R53, R54, R55, R56, R57, R58, R59, R6, R60, R61, R62, R63, R64, R65, R66, R67, R68, R69, R7, R70, R71, R72, R73, R74, R75, R76, R77, R78, R79, R8, R80, R81, R82, R83, R84, R85, R86, R87, R88, R89, R9, R90, R91, R92, R93, R94, R95, R96, R97, R98, R99: value 150 -> 47; footprint Resistor_SMD:R_0201_0603Metric_Pad0.64x0.40mm_HandSolder -> Resistor_SMD:R_0603_1608Metric
